Commit message: ✨ feat(all): 更新模型数据，以 3d 结构设计为准进行优化。

File: MeArm-3D/robot-package/mearm-v1/urdf/mearm-v1.urdf (robot description, URDF)
Before this commit: robot mearm, 7 links, 6 joints
Links:
- link base_link: mass 0.08 -> 0.0266; geometry collision box size=0.047 0.041 0.01; visual box size=0.0228 0.0122 0.0225
- link column_link: mass 0.056 -> 0.0336; geometry collision capsule length=0.012 radius=0.014; visual box size=0.0228 0.0122 0.0225

Commit message: 🐛 fix(all): 夹爪方向反了（D80）+ 消除忙等丢字节 + 精简 memory/skills
## 一、夹爪真机方向修正（ADR D80）

真机实测：S6=40 张开、S6=130 闭合，而原标定 servo = θ + 40 把方向搞反
（网页点「张开」机械爪反而闭合）。修正为 servo = -θ + 140，限位由舵机硬限位
40..130 反算得 gripper.limit 10..100。三端点自洽：
θ=10→S6=130 闭合 / θ=50→S6=90(HOME) / θ=100→S6=40 张开。

⚠️ 不能只翻 reverse：homePose 与关节限位必须一并由舵机硬限位反算。

- robot.yaml：S6 标定 offset 140 / reverse true，gripper.limit 10..100
- 连锁重生成：mearm-v1.urdf、mearm.xml、baseline-kinematics-physics.json
- 黄金数据重采集：fk/ik/joint/sim2sim/workspace 5 份 cases
- 修正写死旧值的断言：calibration/robotModel/robotStore 单测 + Go serial/robot 测试
- 同步文档：decisions.md(D80) / hardware-measurement.md / serial-v1.md
  / coordinate-system.md / ARCHITECTURE_ANALYSIS.md

## 二、固件：消除忙等丢字节路径（修任务④）

上一轮只把 RX 环 64→256 只是把「多久会满」推后，**没消除根因** —— 一条并发路径：
  ① 主循环发 ACK 走 uart_putc，内里 while(tx_full()) 忙等
  ② 忙等期间 cmd_poll() 不执行 ⇒ 停止读 RX 环
  ③ 但 RXCIE0 仍触发、仍写环 ⇒ 环满即静默丢字节
  ④ 丢的若是 SET 6 的字节 ⇒ 该行残缺 ⇒ 解析失败 ⇒ ACK 永不到达
  ⑤ 后端 600ms 超时 ⇒ 表现为「gripper 偶发不执行」

- TX 环 128→256，让多数输出瞬间入队、忙等窗口≈0
- ★ 新增 rx_drop / tx_drop 饱和计数：环满不再静默，可用 STATS 读出
  （这是本次修复的可判定性来源 —— 丢字节原本没有任何外部信号）
- cmd.c 增加 STATS 命令；README 同步

验收：零警告 · FLASH 12848B / RAM 844B · 烧录 COM18 verified ·
压测 240/240 ×2 场景 ×2 轮零缺失 rx_drop=0 · pytest 198 passed ·
test_baseline_frozen 11 passed · 黄金数据 4 份逐位一致 ·
前端 tsc 0 / vitest 401 passed · go test ./... 全绿

## 三、新增诊断工具

probe_gripper_link.py（度量缺陷已修，含误判复盘）· probe_gripper_ws.py（WS 旁听）
· watch_gripper_live.py（轮询 /healthz）。三者为一次性探针，保留供后续复现。

## 四、memory 精简（注入阈值约束）

MEMORY.md 7541 → 3172（阈值 ≈6.3k，超出会被静默截断）；playbook.md 新增 §13
承接搬下来的细节：改真值的连锁清单（D80 实践）、已放弃的路线、夹爪标定实录。
含一次自我纠错：修正臆造字段 is_configured → 实为 is_generated
（content_hash.py:178）。

File: MeArm-3D/robot-package/mearm-v1/urdf/mearm-v1.urdf (robot description, URDF)
Before this commit: robot mearm, 7 links, 6 joints
Joints:
- joint gripper: limit lower=0 upper=1.57079633 effort=0.1765 velocity=10 -> lower=0.174532925 upper=1.74532925 effort=0.1765 velocity=10
